Commit message: add comment

File: resources/robots/a1/urdf/a1.urdf (robot description, URDF)
Before this commit: robot a1_description, 23 links, 22 joints
Links:
- removed link FL_thigh_shoulder
- removed link FR_thigh_shoulder
- removed link RL_thigh_shoulder
- removed link RR_thigh_shoulder
- removed link imu_link
- removed link trunk
- link base: mass None -> 4.713; geometry collision box size=0.267 0.194 0.114; visual mesh filename=../meshes/trunk.dae scale=1 1 1
Joints:
- removed joint FL_hip_fixed
- removed joint FR_hip_fixed
- removed joint RL_hip_fixed
- removed joint RR_hip_fixed
- removed joint floating_base
- removed joint imu_joint
- joint FL_hip_joint: parent trunk -> base
- joint FR_hip_joint: parent trunk -> base
- joint RL_hip_joint: parent trunk -> base
- joint RR_hip_joint: parent trunk -> base
