Commit message: 基本没问题的一版

File: resources/robots/lion/urdf/lion1.urdf (robot description, URDF)
Before this commit: robot lion, 17 links, 16 joints
Links:
- link LegFL_hip: mass 0.39498 -> 0.5; geometry visual mesh filename=../meshes/hip_Link.STL
- link LegFL_thigh: mass 0.5 -> 0.66304
- link LegFR_hip: mass 0.39498 -> 0.5; geometry visual mesh filename=../meshes/hip_Link.STL
- link LegFR_thigh: mass 0.5 -> 0.66304
- link LegHL_hip: mass 0.39498 -> 0.5; geometry visual mesh filename=../meshes/hip_Link.STL
- link LegHL_thigh: mass 0.5 -> 0.66304
- link LegHR_hip: mass 0.39498 -> 0.5; geometry visual mesh filename=../meshes/hip_Link.STL
- link LegHR_thigh: mass 0.5 -> 0.66304
Joints:
- joint JointFL_foot: axis 0 0 1 -> (none)
- joint JointFR_foot: axis 0 0 1 -> (none)
- joint JointHL_foot: axis 0 0 1 -> (none)
- joint JointHR_foot: axis 0 0 1 -> (none)
