Commit message: 更新urdf

File: resources/robots/lion/urdf/lion.urdf (robot description, URDF)
Before this commit: robot lion, 17 links, 16 joints
Links:
- removed link LegFL_foot
- removed link LegFR_foot
- removed link LegHL_foot
- removed link LegHR_foot
- link LegFL_hip: mass 0.39498 -> 1.095; geometry collision mesh filename=../meshes/hip_link.STL; visual mesh filename=../meshes/hip_link.STL
- link LegFL_shank: mass 0.072713 -> 0.233; geometry collision mesh filename=../meshes/shank_link.STL; visual mesh filename=../meshes/shank_link.STL
- link LegFL_thigh: mass 0.5 -> 1.556; geometry collision mesh filename=../meshes/thigh_link.STL; visual mesh filename=../meshes/thigh_link.STL
- link LegFR_hip: mass 0.39498 -> 1.095; geometry collision mesh filename=../meshes/hip_link.STL; visual mesh filename=../meshes/hip_link.STL
- link LegFR_shank: mass 0.072713 -> 0.233; geometry collision mesh filename=../meshes/shank_link.STL; visual mesh filename=../meshes/shank_link.STL
- link LegFR_thigh: mass 0.5 -> 1.556; geometry collision mesh filename=../meshes/thigh_link.STL; visual mesh filename=../meshes/thigh_link.STL
- link LegHL_hip: mass 0.39498 -> 1.095; geometry collision mesh filename=../meshes/hip_link.STL; visual mesh filename=../meshes/hip_link.STL
- link LegHL_shank: mass 0.072713 -> 0.233; geometry collision mesh filename=../meshes/shank_link.STL; visual mesh filename=../meshes/shank_link.STL
- link LegHL_thigh: mass 0.5 -> 1.556; geometry collision mesh filename=../meshes/thigh_link.STL; visual mesh filename=../meshes/thigh_link.STL
- link LegHR_hip: mass 0.39498 -> 1.095; geometry collision mesh filename=../meshes/hip_link.STL; visual mesh filename=../meshes/hip_link.STL
- link LegHR_shank: mass 0.072713 -> 0.233; geometry collision mesh filename=../meshes/shank_link.STL; visual mesh filename=../meshes/shank_link.STL
- link LegHR_thigh: mass 0.5 -> 1.556; geometry collision mesh filename=../meshes/thigh_link.STL; visual mesh filename=../meshes/thigh_link.STL
- link base_link: mass 4 -> 8.286
Joints:
- removed joint JointFL_foot
- removed joint JointFR_foot
- removed joint JointHL_foot
- removed joint JointHR_foot
- joint JointFL_abad: limit lower=-1.0 upper=1.0 effort=55 velocity=30 -> lower=-1 upper=1 effort=30 velocity=20; origin xyz=0.2467 0.09 0 rpy=3.141592653589793 0.0 0  -> xyz=0.2467 0.09 0.0005 rpy=3.141592653589793 0.0 0
- joint JointFL_hip: limit lower=-3.0 upper=3.0 effort=55 velocity=30 -> lower=-2 upper=2 effort=30 velocity=20; type revolute -> continuous
- joint JointFL_knee: limit lower=-3.0 upper=3.0 effort=55 velocity=30 -> lower=-3 upper=3 effort=30 velocity=20; origin xyz=0 0 -0.3 rpy=0 0 0 -> xyz=0 -0.119 -0.3 rpy=0 0 0; type revolute -> continuous
- joint JointFR_abad: limit lower=-1.0 upper=1.0 effort=55 velocity=30 -> lower=-1 upper=1 effort=30 velocity=20; origin xyz=0.2467 -0.09 0 rpy=0.0 0.0 0  -> xyz=0.2467 -0.09 0.0005 rpy=0.0 0.0 0
- joint JointFR_hip: limit lower=-3.0 upper=3.0 effort=55 velocity=30 -> lower=-2 upper=2 effort=30 velocity=20; type revolute -> continuous
- joint JointFR_knee: limit lower=-3.0 upper=3.0 effort=55 velocity=30 -> lower=-3 upper=3 effort=30 velocity=20; origin xyz=0 0 -0.3 rpy=0 0 0 -> xyz=0 -0.119 -0.3 rpy=0 0 0; type revolute -> continuous
- joint JointHL_abad: limit lower=-1.0 upper=1.0 effort=55 velocity=30 -> lower=-1 upper=1 effort=30 velocity=20; origin xyz=-0.2467 0.09 0 rpy=3.141592653589793 3.141592653589793 0  -> xyz=-0.2467 0.09 0.0005 rpy=3.141592653589793 3.141592653589793 0
- joint JointHL_hip: limit lower=-3.0 upper=3.0 effort=55 velocity=30 -> lower=-2 upper=2 effort=30 velocity=20; type revolute -> continuous
- joint JointHL_knee: limit lower=-3.0 upper=3.0 effort=55 velocity=30 -> lower=-3 upper=3 effort=30 velocity=20; origin xyz=0 0 -0.3 rpy=0 0 0 -> xyz=0 -0.119 -0.3 rpy=0 0 0; type revolute -> continuous
- joint JointHR_abad: limit lower=-1.0 upper=1.0 effort=55 velocity=30 -> lower=-1 upper=1 effort=30 velocity=20; origin xyz=-0.2467 -0.09 0 rpy=0.0 3.141592653589793 0  -> xyz=-0.2467 -0.09 0.0005 rpy=0.0 3.141592653589793 0
- joint JointHR_hip: limit lower=-3.0 upper=3.0 effort=55 velocity=30 -> lower=-2 upper=2 effort=30 velocity=20; type revolute -> continuous
- joint JointHR_knee: limit lower=-3.0 upper=3.0 effort=55 velocity=30 -> lower=-3 upper=3 effort=30 velocity=20; origin xyz=0 0 -0.3 rpy=0 0 0 -> xyz=0 -0.119 -0.3 rpy=0 0 0; type revolute -> continuous

Commit message: 新urdf模型可以训练出正常行走

File: resources/robots/lion/urdf/lion.urdf (robot description, URDF)
Before this commit: robot lion, 13 links, 12 joints
Joints:
- joint JointFL_hip: type continuous -> revolute
- joint JointFL_knee: type continuous -> revolute
- joint JointFR_hip: type continuous -> revolute
- joint JointFR_knee: type continuous -> revolute
- joint JointHL_hip: type continuous -> revolute
- joint JointHL_knee: type continuous -> revolute
- joint JointHR_hip: type continuous -> revolute
- joint JointHR_knee: type continuous -> revolute

Commit message: 限制转速为24V时的17

File: resources/robots/lion/urdf/lion.urdf (robot description, URDF)
Before this commit: robot lion, 13 links, 12 joints
Joints:
- joint JointFL_abad: limit lower=-1 upper=1 effort=30 velocity=20 -> lower=-1 upper=1 effort=30 velocity=17
- joint JointFL_hip: limit lower=-2 upper=2 effort=30 velocity=20 -> lower=-2 upper=2 effort=30 velocity=17
- joint JointFL_knee: limit lower=-3 upper=3 effort=30 velocity=20 -> lower=-3 upper=3 effort=30 velocity=17
- joint JointFR_abad: limit lower=-1 upper=1 effort=30 velocity=20 -> lower=-1 upper=1 effort=30 velocity=17
- joint JointFR_hip: limit lower=-2 upper=2 effort=30 velocity=20 -> lower=-2 upper=2 effort=30 velocity=17
- joint JointFR_knee: limit lower=-3 upper=3 effort=30 velocity=20 -> lower=-3 upper=3 effort=30 velocity=17
- joint JointHL_abad: limit lower=-1 upper=1 effort=30 velocity=20 -> lower=-1 upper=1 effort=30 velocity=17
- joint JointHL_hip: limit lower=-2 upper=2 effort=30 velocity=20 -> lower=-2 upper=2 effort=30 velocity=17
- joint JointHL_knee: limit lower=-3 upper=3 effort=30 velocity=20 -> lower=-3 upper=3 effort=30 velocity=17
- joint JointHR_abad: limit lower=-1 upper=1 effort=30 velocity=20 -> lower=-1 upper=1 effort=30 velocity=17
- joint JointHR_hip: limit lower=-2 upper=2 effort=30 velocity=20 -> lower=-2 upper=2 effort=30 velocity=17
- joint JointHR_knee: limit lower=-3 upper=3 effort=30 velocity=20 -> lower=-3 upper=3 effort=30 velocity=17

Commit message: 修改碰撞模型训练

File: resources/robots/lion/urdf/lion.urdf (robot description, URDF)
Before this commit: robot lion, 13 links, 12 joints
Links:
- link LegFL_hip: geometry visual mesh filename=../meshes/hip_link.STL
- link LegFL_thigh: geometry visual mesh filename=../meshes/thigh_link.STL
- link LegFR_hip: geometry visual mesh filename=../meshes/hip_link.STL
- link LegFR_thigh: geometry visual mesh filename=../meshes/thigh_link.STL
- link LegHL_hip: geometry visual mesh filename=../meshes/hip_link.STL
- link LegHL_thigh: geometry visual mesh filename=../meshes/thigh_link.STL
- link LegHR_hip: geometry visual mesh filename=../meshes/hip_link.STL
- link LegHR_thigh: geometry visual mesh filename=../meshes/thigh_link.STL
Joints:
- joint JointFL_abad: limit lower=-1 upper=1 effort=30 velocity=20 -> lower=-1 upper=1 effort=30 velocity=17
- joint JointFL_hip: limit lower=-2 upper=2 effort=30 velocity=20 -> lower=-2 upper=2 effort=30 velocity=17
- joint JointFL_knee: limit lower=-3 upper=3 effort=30 velocity=20 -> lower=-3 upper=3 effort=30 velocity=17
- joint JointFR_abad: limit lower=-1 upper=1 effort=30 velocity=20 -> lower=-1 upper=1 effort=30 velocity=17
- joint JointFR_hip: limit lower=-2 upper=2 effort=30 velocity=20 -> lower=-2 upper=2 effort=30 velocity=17
- joint JointFR_knee: limit lower=-3 upper=3 effort=30 velocity=20 -> lower=-3 upper=3 effort=30 velocity=17
- joint JointHL_abad: limit lower=-1 upper=1 effort=30 velocity=20 -> lower=-1 upper=1 effort=30 velocity=17
- joint JointHL_hip: limit lower=-2 upper=2 effort=30 velocity=20 -> lower=-2 upper=2 effort=30 velocity=17
- joint JointHL_knee: limit lower=-3 upper=3 effort=30 velocity=20 -> lower=-3 upper=3 effort=30 velocity=17
- joint JointHR_abad: limit lower=-1 upper=1 effort=30 velocity=20 -> lower=-1 upper=1 effort=30 velocity=17
- joint JointHR_hip: limit lower=-2 upper=2 effort=30 velocity=20 -> lower=-2 upper=2 effort=30 velocity=17
- joint JointHR_knee: limit lower=-3 upper=3 effort=30 velocity=20 -> lower=-3 upper=3 effort=30 velocity=17

Commit message: 给定参考轨迹，训练结果一般

File: resources/robots/lion/urdf/lion.urdf (robot description, URDF)
Before this commit: robot lion, 13 links, 12 joints
Links:
- link LegFL_shank: geometry collision sphere radius=0.02; visual mesh filename=../meshes/shank_link.STL
- link LegFR_shank: geometry collision sphere radius=0.02; visual mesh filename=../meshes/shank_link.STL
- link LegHL_shank: geometry collision sphere radius=0.02; visual mesh filename=../meshes/shank_link.STL
- link LegHR_shank: geometry collision sphere radius=0.02; visual mesh filename=../meshes/shank_link.STL
